File: 9axis.sch (KiCad schematic (older format))
At the start: 4 parts, among them U2 MPU-9250

Commit message: Started changes after first round, micro usb connector, fixing footprint for accelerometer
Parts:
- U2: footprint mpu-9250:MPU-9250 -> Housings_DFN_QFN:QFN-24-1EP_3x3mm_Pitch0.4mm
Changed lines of the file:
@@
 F 0 "U2" H 5650 5337 60  0000 C CNN
 F 1 "MPU-9250" H 5650 5231 60  0000 C CNN
-F 2 "mpu-9250:MPU-9250" H 5650 5000 60  0001 C CNN
+F 2 "Housings_DFN_QFN:QFN-24-1EP_3x3mm_Pitch0.4mm" H 5650 5000 60  0001 C CNN
 F 3 "" H 5650 5000 60  0000 C CNN
 	1    5650 4400
